File: tools/templates/mcp_standard_placements.kicad_sch (KiCad schematic)
At the start: 150 parts, among them J1 ICSP, J3 PIR BOARD, J5 MOTOR, J6 DNP, Q1 FMOS3401A?, Q11 MMBTA55?, Q2 BC847B?, Q3 MMBTA55?, Q4 MMBTA55?, Q5 MMBTA55?, Q6 MMBTA55?, Q7 BC857C?, Q8 N/P pair? (372A), Q9 DNP, U1 S-1200B45? [pins], U106 U6A / DNP, U2 SN74LVC2G14DBV?, U3 SGM8542XS, U4 PIC16F18855, U5 MX512H, U6 S-812C33AMC? / 3.3V, U7 DNP, Y1 20 MHz

Commit message: Resolve C26 to PIC RA1 from annotated board photo
Parts:
- C25, C26, U4: ConnectionEvidence (none) -> v0.9.17 user-annotated photo: C25 right pad/model1 -> PIC2/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
Other:
- moved on the sheet: C25, C26, C39
Changed lines of the file:
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@@
 				(font
 					(size 1.27 1.27)
-				) (hide yes))
+				)
+				(hide yes)
+			)
+		)
+		(property "MeasurementEvidence" "v0.9.16 CORRECTION: user confirms PIC21/RB0 -> TP16 -> Q2 single pad; TP16-VREF = 0.8 Mohm. User explicitly withdraws PIC21-VREF. PIC21/V026 belongs to H_PIR_SIG, separate from VREF. RA2/V035 and R21/V071 remain VREF. This supersedes every earlier RB0/V026-to-VREF statement."
+			(at 262.89 78.74 0)
+			(effects
+				(font
+					(size 1.27 1.27)
+				)
+				(hide yes)
+			)
+		)
+		(property "ConnectionEvidence" "v0.9.17 user-annotated photo: C25 right pad/model1 -> PIC2/RA0; C26 right pad/model1 -> PIC3/RA1. Left pads/model2 are common, retaining earlier V029-GND evidence. No new numeric resistance or capacitance supplied. C26 joins the existing RA1/R28/R29/TP7 net, separate from RA0 and VREF."
+			(at 262.89 78.74 0)
+			(effects
+				(font
+					(size 1.27 1.27)
+				)
+				(hide yes)
+			)
 		)
-    (property "MeasurementEvidence" "v0.9.16 CORRECTION: user confirms PIC21/RB0 -> TP16 -> Q2 single pad; TP16-VREF = 0.8 Mohm. User explicitly withdraws PIC21-VREF. PIC21/V026 belongs to H_PIR_SIG, separate from VREF. RA2/V035 and R21/V071 remain VREF. This supersedes every earlier RB0/V026-to-VREF statement." (at 262.89 78.74 0)
-      (effects (font (size 1.27 1.27)) (hide yes))
-    )
 		(pin "1"
 		)
@@
 	(symbol
 		(lib_id "Device:C")
-		(at 312.42 62.23 0)
+		(at 322.58 78.74 0)
 		(unit 1)
 		(body_style 1)
@@
 		(dnp no)
 		(property "Reference" "C25"
-			(at 313.05500000000006 64.77 0)
+			(at 323.21500000000003 81.28 0)
 			(show_name no)
 			(do_not_autoplace no)
@@
 		)
 		(property "Value" "?"
-			(at 313.05500000000006 59.69 0)
+			(at 323.21500000000003 76.19999999999999 0)
 			(show_name no)
 			(do_not_autoplace no)
@@
 		)
 		(property "Footprint" "Capacitor_SMD:C_0805_2012Metric"
-			(at 313.385 58.42 0)
+			(at 323.54499999999996 74.93 0)
 			(hide yes)
 			(show_name no)
@@
 		)
 		(property "Datasheet" ""
-			(at 312.42 62.23 0)
+			(at 322.58 78.74 0)
 			(hide yes)
 			(show_name no)
@@
 		)
 		(property "Description" "Unpolarized capacitor"
-			(at 312.42 62.23 0)
+			(at 322.58 78.74 0)
 			(hide yes)
 			(show_name no)
@@
 			)
 		)
+		(property "ConnectionEvidence" "v0.9.17 user-annotated photo: C25 right pad/model1 -> PIC2/RA0; C26 right pad/model1 -> PIC3/RA1. Left pads/model2 are common, retaining earlier V029-GND evidence. No new numeric resistance or capacitance supplied. C26 joins the existing RA1/R28/R29/TP7 net, separate from RA0 and VREF."
+			(at 322.58 78.74 0)
+			(effects
+				(font
+					(size 1.27 1.27)
+				)
+				(hide yes)
+			)
+		)
 		(pin "1"
 		)
@@
 	(symbol
 		(lib_id "Device:C")
-		(at 224.79 48.26 0)
+		(at 312.42 78.74 0)
 		(unit 1)
 		(body_style 1)
@@
 		(dnp no)
 		(property "Reference" "C26"
-			(at 225.425 50.8 0)
+			(at 313.05500000000006 81.28 0)
 			(show_name no)
 			(do_not_autoplace no)
@@
 		)
 		(property "Value" "?"
-			(at 225.425 45.72 0)
+			(at 313.05500000000006 76.19999999999999 0)
 			(show_name no)
 			(do_not_autoplace no)
@@
 		)
 		(property "Footprint" "Capacitor_SMD:C_0805_2012Metric"
-			(at 225.755 44.45 0)
+			(at 313.385 74.93 0)
 			(hide yes)
 			(show_name no)
@@
 		)
 		(property "Datasheet" ""
-			(at 224.79 48.26 0)
+			(at 312.42 78.74 0)
 			(hide yes)
 			(show_name no)
@@
 		)
 		(property "Description" "Unpolarized capacitor"
-			(at 224.79 48.26 0)
+			(at 312.42 78.74 0)
 			(hide yes)
 			(show_name no)
@@
 			)
 		)
+		(property "ConnectionEvidence" "v0.9.17 user-annotated photo: C25 right pad/model1 -> PIC2/RA0; C26 right pad/model1 -> PIC3/RA1. Left pads/model2 are common, retaining earlier V029-GND evidence. No new numeric resistance or capacitance supplied. C26 joins the existing RA1/R28/R29/TP7 net, separate from RA0 and VREF."
+			(at 312.42 78.74 0)
+			(effects
+				(font
+					(size 1.27 1.27)
+				)
+				(hide yes)
+			)
+		)
 		(pin "1"
 		)
@@
 	(symbol
 		(lib_id "Device:C")
-		(at 300.99 67.31 0)
+		(at 300.99 78.74 0)
 		(unit 1)
 		(body_style 1)
@@
 		(dnp no)
 		(property "Reference" "C39"
-			(at 301.625 69.85 0)
+			(at 301.625 81.27999999999999 0)
 			(show_name no)
 			(do_not_autoplace no)
@@
 		)
 		(property "Value" "?"
-			(at 301.625 64.77000000000001 0)
+			(at 301.625 76.2 0)
 			(show_name no)
 			(do_not_autoplace no)
@@
 		)
 		(property "Footprint" "Capacitor_SMD:C_0805_2012Metric"
-			(at 301.95500000000004 63.50000000000001 0)
+			(at 301.95500000000004 74.93 0)
 			(hide yes)
 			(show_name no)
@@
 		)
 		(property "Datasheet" ""
-			(at 300.99 67.31 0)
+			(at 300.99 78.74 0)
 			(hide yes)
 			(show_name no)
@@
 		)
 		(property "Description" "Unpolarized capacitor"
-			(at 300.99 67.31 0)
+			(at 300.99 78.74 0)
 			(hide yes)
 			(show_name no)
@@
 		)
 		(property "ViaEvidence" "v0.9.9: User checked V035-VREF TP. Prior photo association V035-PIC4/RA2-C39.1 retained; joins the already confirmed RB0/V026/R21.2/V071 VREF node. No voltage or numerical resistance supplied. Other modeled bias branches retain earlier inferred status."
-			(at 300.99 67.31 0)
+			(at 300.99 78.74 0)
 			(effects
 				(font
@@
 				(font
 					(size 1.27 1.27)
-				) (hide yes))
+				)
+				(hide yes)
+			)
+		)
+		(property "MeasurementEvidence" "v0.9.16 CORRECTION: user confirms PIC21/RB0 -> TP16 -> Q2 single pad; TP16-VREF = 0.8 Mohm. User explicitly withdraws PIC21-VREF. PIC21/V026 belongs to H_PIR_SIG, separate from VREF. RA2/V035 and R21/V071 remain VREF. This supersedes every earlier RB0/V026-to-VREF statement."
+			(at 356.87 223.52 0)
+			(effects
+				(font
+					(size 1.27 1.27)
+				)
+				(hide yes)
+			)
 		)
-    (property "MeasurementEvidence" "v0.9.16 CORRECTION: user confirms PIC21/RB0 -> TP16 -> Q2 single pad; TP16-VREF = 0.8 Mohm. User explicitly withdraws PIC21-VREF. PIC21/V026 belongs to H_PIR_SIG, separate from VREF. RA2/V035 and R21/V071 remain VREF. This supersedes every earlier RB0/V026-to-VREF statement." (at 356.87 223.52 0)
-      (effects (font (size 1.27 1.27)) (hide yes))
-    )
 		(pin "1"
 		)
@@
 				(font
 					(size 1.27 1.27)
-				) (hide yes))
+				)
+				(hide yes)
+			)
+		)
+		(property "MeasurementEvidence" "v0.9.16 CORRECTION: user confirms PIC21/RB0 -> TP16 -> Q2 single pad; TP16-VREF = 0.8 Mohm. User explicitly withdraws PIC21-VREF. PIC21/V026 belongs to H_PIR_SIG, separate from VREF. RA2/V035 and R21/V071 remain VREF. This supersedes every earlier RB0/V026-to-VREF statement."
+			(at 307.34 229.87 0)
+			(effects
+				(font
+					(size 1.27 1.27)
+				)
+				(hide yes)
+			)
 		)
-    (property "MeasurementEvidence" "v0.9.16 CORRECTION: user confirms PIC21/RB0 -> TP16 -> Q2 single pad; TP16-VREF = 0.8 Mohm. User explicitly withdraws PIC21-VREF. PIC21/V026 belongs to H_PIR_SIG, separate from VREF. RA2/V035 and R21/V071 remain VREF. This supersedes every earlier RB0/V026-to-VREF statement." (at 307.34 229.87 0)
-      (effects (font (size 1.27 1.27)) (hide yes))
-    )
 		(pin "1"
 		)
@@
 				(font
 					(size 1.27 1.27)
-				) (hide yes))
+				)
+				(hide yes)
+			)
 		)
 		(property "MeasurementEvidence" "v0.9.16 CORRECTION: user confirms PIC21/RB0 -> TP16 -> Q2 single pad; TP16-VREF = 0.8 Mohm. User explicitly withdraws PIC21-VREF. PIC21/V026 belongs to H_PIR_SIG, separate from VREF. RA2/V035 and R21/V071 remain VREF. This supersedes every earlier RB0/V026-to-VREF statement."
@@
 				(font
 					(size 1.27 1.27)
-				) (hide yes))
+				)
+				(hide yes)
+			)
 		)
 		(pin "1"
@@
 				(font
 					(size 1.27 1.27)
-				) (hide yes))
+				)
+				(hide yes)
+			)
+		)
+		(property "ViaEvidence" "v0.9.16 CORRECTION: user confirms PIC21/RB0 -> TP16 -> Q2 single pad; TP16-VREF = 0.8 Mohm. User explicitly withdraws PIC21-VREF. PIC21/V026 belongs to H_PIR_SIG, separate from VREF. RA2/V035 and R21/V071 remain VREF. This supersedes every earlier RB0/V026-to-VREF statement."
+			(at 379.73 335.28 0)
+			(effects
+				(font
+					(size 1.27 1.27)
+				)
+				(hide yes)
+			)
 		)
-    (property "ViaEvidence" "v0.9.16 CORRECTION: user confirms PIC21/RB0 -> TP16 -> Q2 single pad; TP16-VREF = 0.8 Mohm. User explicitly withdraws PIC21-VREF. PIC21/V026 belongs to H_PIR_SIG, separate from VREF. RA2/V035 and R21/V071 remain VREF. This supersedes every earlier RB0/V026-to-VREF statement." (at 379.73 335.28 0)
-      (effects (font (size 1.27 1.27)) (hide yes))
-    )
 		(pin "1"
 		)
@@
 				(font
 					(size 1.27 1.27)
-				) (hide yes))
+				)
+				(hide yes)
+			)
+		)
+		(property "MeasurementEvidence" "v0.9.16 CORRECTION: user confirms PIC21/RB0 -> TP16 -> Q2 single pad; TP16-VREF = 0.8 Mohm. User explicitly withdraws PIC21-VREF. PIC21/V026 belongs to H_PIR_SIG, separate from VREF. RA2/V035 and R21/V071 remain VREF. This supersedes every earlier RB0/V026-to-VREF statement."
+			(at 478.79 382.27 0)
+			(effects
+				(font
+					(size 1.27 1.27)
+				)
+				(hide yes)
+			)
 		)
-    (property "MeasurementEvidence" "v0.9.16 CORRECTION: user confirms PIC21/RB0 -> TP16 -> Q2 single pad; TP16-VREF = 0.8 Mohm. User explicitly withdraws PIC21-VREF. PIC21/V026 belongs to H_PIR_SIG, separate from VREF. RA2/V035 and R21/V071 remain VREF. This supersedes every earlier RB0/V026-to-VREF statement." (at 478.79 382.27 0)
-      (effects (font (size 1.27 1.27)) (hide yes))
-    )
 		(pin "1"
 		)

Commit message: Reconstruct C6 in parallel with C5 from board photos
Parts:
- C5, C6: ConnectionEvidence (none) -> v0.9.18: C6 is reconstructed in parallel with C5 from the u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
Changed lines of the file:
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@@
 			)
 		)
+    (property "ConnectionEvidence" "v0.9.18: C6 is reconstructed in parallel with C5 from the user proposal and photos IMG_2431/IMG_2432. C6 upper pad/model1 joins the C5-positive supply copper (H_RF_VDD, after L1); lower pad/model2 joins GND. Photo-supported, not a new meter-confirmed connection. C6 capacitance remains unknown. Earlier 400 kohm output exclusion and 10 ohm Q8-supply-path reading are retained; the latter does not independently prove Q8 source wiring." (at 237.49 181.61 0)
+      (effects (font (size 1.27 1.27)) (hide yes))
+    )
 		(pin "1"
 		)
@@
 			)
 		)
+    (property "ConnectionEvidence" "v0.9.18: C6 is reconstructed in parallel with C5 from the user proposal and photos IMG_2431/IMG_2432. C6 upper pad/model1 joins the C5-positive supply copper (H_RF_VDD, after L1); lower pad/model2 joins GND. Photo-supported, not a new meter-confirmed connection. C6 capacitance remains unknown. Earlier 400 kohm output exclusion and 10 ohm Q8-supply-path reading are retained; the latter does not independently prove Q8 source wiring." (at 259.08 181.61 0)
+      (effects (font (size 1.27 1.27)) (hide yes))
+    )
 		(pin "1"
 		)
