File: tools/templates/mcp_standard_placements.kicad_sch (KiCad schematic)
At the start: 149 parts, among them J1 ICSP, J3 PIR BOARD, J5 MOTOR, J6 DNP, Q1 FMOS3401A?, Q11 MMBTA55?, Q2 BC847B?, Q3 MMBTA55?, Q4 MMBTA55?, Q5 MMBTA55?, Q6 MMBTA55?, Q7 BC857C?, Q8 N/P pair? (372A), Q9 NPN option / DNP, U1 S-1200B45? [pins], U106 U6A / LDO option, U2 SN74LVC2G14DBV?, U3 SGM8542XS, U4 PIC16F18855, U5 MX512H, U6 S-812C33AMC? / 3.3V, U7 DNP, Y1 20 MHz

Commit message: Connect rear C49 between ANT2 and ground
Parts:
- C49: ConnectionEvidence (none) -> User confirms C49 connects between ANT2 and GND (2026-10-09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; LocationEvidence Clearly visible empty C49 on rear IMG_2442.jpg beside anten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 -> Rear C49 footprint beside antenna wire terminations in IMG_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
Changed lines of the file:
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@@
 			)
 		)
-		(property "LocationEvidence" "Clearly visible empty C49 on rear IMG_2442.jpg beside antenna wire terminations. Retained; both copper destinations unresolved."
+		(property "LocationEvidence" "Rear C49 footprint beside antenna wire terminations in IMG_2442.jpg; presence confirmed by user 2026-10-09. Existing DNP population retained."
 			(at 259.08 379.73 0)
 			(effects
@@
 			)
 		)
+(property "ConnectionEvidence" "User confirms C49 connects between ANT2 and GND (2026-10-09). Model pin1 = H_ANT_B / ANT2, pin2 = GND. Nonpolar capacitor: pin numbering is a schematic convention, not a separately measured physical pad orientation. No capacitance value or population change reported." (at 259.08 379.73 0)
+(effects (font (size 1.27 1.27)) (hide yes))
+)
 		(pin "1"
 		)

Commit message: Clean up current schematic evidence and finishing plan for v0.9.29
Parts:
- C27: CurrentEvidence (none) -> Motor supply bypass across VSYS (U5 pin4 supply) and GND fr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
- C35: CurrentEvidence (none) -> Unknown capacitance. Model2/upper end is GND/S1 upper-right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
- C49: CurrentEvidence (none) -> Rear C49 footprint beside antenna wire terminations in IMG_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
- C5: CurrentEvidence (none) -> User confirms radial electrolytic C5, 6.33 mm diameter and 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
- D2: CurrentEvidence (none) -> 4P exact identity unresolved. In-circuit diode readings sup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
- D3: CurrentEvidence (none) -> A7 and the series-dual pin map support BAV99. User confirms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
- D4, D5: CurrentEvidence (none) -> 5U supports an SD05 TVS candidate. Model1/cathode reaches I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
- D6: CurrentEvidence (none) -> G3 marking; user measurements establish anode at GND, catho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
- J3: CurrentEvidence (none) -> PIR connector: pin1 supply; pin2 to R38 K/right/model1 at 1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
- L1: CurrentEvidence (none) -> User LCR-meter reading: L1 = 1.4 uH. Test frequency, test m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
- L2: CurrentEvidence (none) -> User LCR-meter reading: L2 = 2.2 uH. Test frequency, test m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
- LED1: CurrentEvidence (none) -> User confirms square 1.5 x 1.5 mm package containing red an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
- Q1: CurrentEvidence (none) -> R1A marking matches Formosa FMOS3401A datasheet p5; SOT-23 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
- Q2: CurrentEvidence (none) -> 1FW supports BC847B. Candidate B=R, E=L, C=S and interface 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
- Q7: CurrentEvidence (none) -> 3GW supports BC857C PNP. Photo and 11.2 kohm R18+R19 path s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
- Q8: CurrentEvidence (none) -> 3724A supports the SIL3724A complementary MOSFET candidate;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
- Q9: CurrentEvidence (none) -> v0.9.24: use generic NPN BEC symbol for empty Q9, consisten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
- R37: CurrentEvidence (none) -> 22 ohm from marking. Input/model1 joins printed VDD through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
- R39: CurrentEvidence (none) -> 10k from marking. Model2 joins printed VDD through V063/V06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
- R40: CurrentEvidence (none) -> 10k from marking, between ICSP_DAT/PIC28 and H_BUTTON. H_BU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
- R41: CurrentEvidence (none) -> User reads 331: 330 ohm. Model1/right end reaches J1 VPP/MC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
- S1: CurrentEvidence (none) -> Measured body 6 x 6 x 4 mm plus 2 mm actuator. Stock SW_Pus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
- U106: CurrentEvidence (none) -> v0.9.24: same measured/photo-supported U6A input/output/GND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
- U6: CurrentEvidence (none) -> C2NM supports candidate S-812C33AMC: pin1 VSS, pin2 VIN, pi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

Commit message: Resolve RF drive routing from original photos and document review findings
Parts:
- D1, R6, R7, TP3: CurrentEvidence (none) -> v0.9.30 original IMG_2431: TP3/PIC13 common reaches R6 uppe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
- Q11, Q3, Q4, Q5, Q6: CurrentEvidence (none) -> Provisional 2H / MMBTA55 PNP candidate; physical R->base1, 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
Changed lines of the file:
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@@
 			)
 		)
+    (property "CurrentEvidence" "v0.9.30 original IMG_2431: TP3/PIC13 common reaches R6 upper (model2), R7 upper (model1) and D1 single pad/native3. D1 paired-right/native2 joins R7 lower/C9 upper/U2 native1. Photo-supported; not new bench readings. BAV99 identity and RF timing remain candidates." (at 38.1 222.25 0)
+      (effects (font (size 1.27 1.27)) (hide yes))
+    )
 		(pin "1"
 		)
@@
 			)
 		)
+    (property "CurrentEvidence" "v0.9.30 original IMG_2431: TP3/PIC13 common reaches R6 upper (model2), R7 upper (model1) and D1 single pad/native3. D1 paired-right/native2 joins R7 lower/C9 upper/U2 native1. Photo-supported; not new bench readings. BAV99 identity and RF timing remain candidates." (at 38.1 177.8 0)
+      (effects (font (size 1.27 1.27)) (hide yes))
+    )
 		(pin "1"
 		)
@@
 			)
 		)
+    (property "CurrentEvidence" "v0.9.30 original IMG_2431: TP3/PIC13 common reaches R6 upper (model2), R7 upper (model1) and D1 single pad/native3. D1 paired-right/native2 joins R7 lower/C9 upper/U2 native1. Photo-supported; not new bench readings. BAV99 identity and RF timing remain candidates." (at 49.53 200.66 0)
+      (effects (font (size 1.27 1.27)) (hide yes))
+    )
 		(pin "1"
 		)
@@
 			)
 		)
+    (property "CurrentEvidence" "v0.9.30 original IMG_2431: TP3/PIC13 common reaches R6 upper (model2), R7 upper (model1) and D1 single pad/native3. D1 paired-right/native2 joins R7 lower/C9 upper/U2 native1. Photo-supported; not new bench readings. BAV99 identity and RF timing remain candidates." (at 52.07 251.46 0)
+      (effects (font (size 1.27 1.27)) (hide yes))
+    )
 		(pin "1"
 		)
@@
 			)
 		)
+    (property "CurrentEvidence" "Provisional 2H / MMBTA55 PNP candidate; physical R->base1, L->emitter2/GND, S->collector3 is unverified. This is not ordinary positive-GPIO PNP switching. Preserve copper pending one Q3-cell polarity/orientation test; no NPN substitution by plausibility." (at 50.8 347.98 0)
+      (effects (font (size 1.27 1.27)) (hide yes))
+    )
 		(pin "1"
 		)
@@
 			)
 		)
+    (property "CurrentEvidence" "Provisional 2H / MMBTA55 PNP candidate; physical R->base1, L->emitter2/GND, S->collector3 is unverified. This is not ordinary positive-GPIO PNP switching. Preserve copper pending one Q3-cell polarity/orientation test; no NPN substitution by plausibility." (at 104.14 347.98 0)
+      (effects (font (size 1.27 1.27)) (hide yes))
+    )
 		(pin "1"
 		)
@@
 			)
 		)
+    (property "CurrentEvidence" "Provisional 2H / MMBTA55 PNP candidate; physical R->base1, L->emitter2/GND, S->collector3 is unverified. This is not ordinary positive-GPIO PNP switching. Preserve copper pending one Q3-cell polarity/orientation test; no NPN substitution by plausibility." (at 157.48 347.98 0)
+      (effects (font (size 1.27 1.27)) (hide yes))
+    )
 		(pin "1"
 		)
@@
 			)
 		)
+    (property "CurrentEvidence" "Provisional 2H / MMBTA55 PNP candidate; physical R->base1, L->emitter2/GND, S->collector3 is unverified. This is not ordinary positive-GPIO PNP switching. Preserve copper pending one Q3-cell polarity/orientation test; no NPN substitution by plausibility." (at 210.82 347.98 0)
+      (effects (font (size 1.27 1.27)) (hide yes))
+    )
 		(pin "1"
 		)
@@
 			)
 		)
+    (property "CurrentEvidence" "Provisional 2H / MMBTA55 PNP candidate; physical R->base1, L->emitter2/GND, S->collector3 is unverified. This is not ordinary positive-GPIO PNP switching. Preserve copper pending one Q3-cell polarity/orientation test; no NPN substitution by plausibility." (at 264.16 347.98 0)
+      (effects (font (size 1.27 1.27)) (hide yes))
+    )
 		(pin "1"
 		)

Commit message: Declare power sources and consolidate remaining schematic work
Parts:
- R33: CurrentEvidence (none) -> INVENTORY UNVERIFIED (E07): inherited 10k PIR pull-up. Cite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

Commit message: Record Q3 diode results and withdraw unsupported R33 pull-up
Parts:
- removed R33: 10k, Resistor_SMD:R_0603_1608Metric, symbol Device:R
- J3: CurrentEvidence PIR connector: pin1 supply; pin2 to R38 K/right/model1 at 1 ohm, with 10k through R38; pin3 GND at 1 ohm. The Q2 single-pad/TP16 output reaches PIC21/RB0 by user correction. PIC21-to-VREF was withdrawn after TP16-VREF measured 0.8 Mohm. Q2/R33 device behavior remains qualified. -> PIR connector: pin1 supply; pin2 to R38 K/right/model1 at 1 ohm, with 10k through R38; pin3 GND at 1 ohm. The Q2 single-pad/TP16 output reaches PIC21/RB0 by user correction. PIC21-to-VREF was withdrawn after TP16-VREF measured 0.8 Mohm. Q2 behavior remains unverified; unsupported R33 pull-up withdrawn.
- Q11, Q4, Q5, Q6: CurrentEvidence Provisional 2H / MMBTA55 PNP candidate; physical R->base1, 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 -> Same 2H marking as Q3; PNP type/pinout remains disputed by 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
- Q3: CurrentEvidence Provisional 2H / MMBTA55 PNP candidate; physical R->base1, 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 -> DISPUTED 2H / MMBTA55 PNP candidate. Q3 in-circuit diode re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
- R39: CurrentEvidence 10k from marking. Model2 joins printed VDD through V063/V064; model1 remains on the inferred Q2 base/R38 node. PIR output TP16/Q2.S to PIC21 is confirmed; transistor pin functions and the R33 branch remain qualified. -> 10k from marking. Model2 joins printed VDD through V063/V064; model1 remains on the inferred Q2 base/R38 node. PIR output TP16/Q2.S to PIC21 is confirmed; transistor pin functions remain unverified. Unsupported R33 pull-up withdrawn.
Changed lines of the file:
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@@
 			)
 		)
-		(property "CurrentEvidence" "Provisional 2H / MMBTA55 PNP candidate; physical R->base1, L->emitter2/GND, S->collector3 is unverified. This is not ordinary positive-GPIO PNP switching. Preserve copper pending one Q3-cell polarity/orientation test; no NPN substitution by plausibility."
+		(property "CurrentEvidence" "DISPUTED 2H / MMBTA55 PNP candidate. Q3 in-circuit diode readings: L->R 2.3V, L->S latest 0.48V (earlier 0.35V); reverse directions and R/S both ways OL. These do not confirm B=R/E=L/C=S. Copper and candidate symbol retained pending isolated-device identification; no MOSFET identity inferred from one forward path."
 			(at 50.8 347.98 0)
 			(effects
@@
 			)
 		)
-		(property "CurrentEvidence" "Provisional 2H / MMBTA55 PNP candidate; physical R->base1, L->emitter2/GND, S->collector3 is unverified. This is not ordinary positive-GPIO PNP switching. Preserve copper pending one Q3-cell polarity/orientation test; no NPN substitution by plausibility."
+		(property "CurrentEvidence" "Same 2H marking as Q3; PNP type/pinout remains disputed by Q3 in-circuit diode results (0.48V L->S; 2.3V L->R; other directions OL). This device was not diode-tested. Retain existing copper and provisional PNP symbol pending family identification."
 			(at 104.14 347.98 0)
 			(effects
@@
 			)
 		)
-		(property "CurrentEvidence" "Provisional 2H / MMBTA55 PNP candidate; physical R->base1, L->emitter2/GND, S->collector3 is unverified. This is not ordinary positive-GPIO PNP switching. Preserve copper pending one Q3-cell polarity/orientation test; no NPN substitution by plausibility."
+		(property "CurrentEvidence" "Same 2H marking as Q3; PNP type/pinout remains disputed by Q3 in-circuit diode results (0.48V L->S; 2.3V L->R; other directions OL). This device was not diode-tested. Retain existing copper and provisional PNP symbol pending family identification."
 			(at 157.48 347.98 0)
 			(effects
@@
 			)
 		)
-		(property "CurrentEvidence" "Provisional 2H / MMBTA55 PNP candidate; physical R->base1, L->emitter2/GND, S->collector3 is unverified. This is not ordinary positive-GPIO PNP switching. Preserve copper pending one Q3-cell polarity/orientation test; no NPN substitution by plausibility."
+		(property "CurrentEvidence" "Same 2H marking as Q3; PNP type/pinout remains disputed by Q3 in-circuit diode results (0.48V L->S; 2.3V L->R; other directions OL). This device was not diode-tested. Retain existing copper and provisional PNP symbol pending family identification."
 			(at 210.82 347.98 0)
 			(effects
@@
 			)
 		)
-		(property "CurrentEvidence" "Provisional 2H / MMBTA55 PNP candidate; physical R->base1, L->emitter2/GND, S->collector3 is unverified. This is not ordinary positive-GPIO PNP switching. Preserve copper pending one Q3-cell polarity/orientation test; no NPN substitution by plausibility."
+		(property "CurrentEvidence" "Same 2H marking as Q3; PNP type/pinout remains disputed by Q3 in-circuit diode results (0.48V L->S; 2.3V L->R; other directions OL). This device was not diode-tested. Retain existing copper and provisional PNP symbol pending family identification."
 			(at 264.16 347.98 0)
 			(effects
@@
 			)
 		)
-		(property "CurrentEvidence" "PIR connector: pin1 supply; pin2 to R38 K/right/model1 at 1 ohm, with 10k through R38; pin3 GND at 1 ohm. The Q2 single-pad/TP16 output reaches PIC21/RB0 by user correction. PIC21-to-VREF was withdrawn after TP16-VREF measured 0.8 Mohm. Q2/R33 device behavior remains qualified."
+		(property "CurrentEvidence" "PIR connector: pin1 supply; pin2 to R38 K/right/model1 at 1 ohm, with 10k through R38; pin3 GND at 1 ohm. The Q2 single-pad/TP16 output reaches PIC21/RB0 by user correction. PIC21-to-VREF was withdrawn after TP16-VREF measured 0.8 Mohm. Q2 behavior remains unverified; unsupported R33 pull-up withdrawn."
 			(at 405.13 327.66 0)
 			(effects
@@
 			)
 		)
-		(property "CurrentEvidence" "10k from marking. Model2 joins printed VDD through V063/V064; model1 remains on the inferred Q2 base/R38 node. PIR output TP16/Q2.S to PIC21 is confirmed; transistor pin functions and the R33 branch remain qualified."
+		(property "CurrentEvidence" "10k from marking. Model2 joins printed VDD through V063/V064; model1 remains on the inferred Q2 base/R38 node. PIR output TP16/Q2.S to PIC21 is confirmed; transistor pin functions remain unverified. Unsupported R33 pull-up withdrawn."
 			(at 351.79 355.6 0)
 			(effects
@@
 					(unit 1)
 				)
-			)
-		)
-	)
-	(symbol
-		(lib_id "Device:R")
-		(at 393.7 353.06 0)
-		(unit 1)
-		(body_style 1)
-		(exclude_from_sim no)
-		(in_bom yes)
-		(on_board yes)
-		(in_pos_files yes)
-		(dnp no)
-		(property "Reference" "R33"
-			(at 395.732 353.06 90)
-			(show_name no)
-			(do_not_autoplace no)
-			(effects
-				(font
-					(size 1.27 1.27)
-				)
-			)
-		)
-		(property "Value" "10k"
-			(at 393.7 353.06 90)
-			(show_name no)
-			(do_not_autoplace no)
-			(effects
-				(font
-					(size 1.27 1.27)
-				)
-			)
-		)
-		(property "Footprint" "Resistor_SMD:R_0603_1608Metric"
-			(at 391.922 353.06 90)
-			(hide yes)
-			(show_name no)
-			(do_not_autoplace no)
-			(effects
-				(font
-					(size 1.27 1.27)
-				)
-			)
-		)
-		(property "Datasheet" ""
-			(at 393.7 353.06 0)
-			(hide yes)
-			(show_name no)
-			(do_not_autoplace no)
-			(effects
-				(font
-					(size 1.27 1.27)
-				)
-			)
-		)
-		(property "Description" "Resistor"
-			(at 393.7 353.06 0)
-			(hide yes)
-			(show_name no)
-			(do_not_autoplace no)
-			(effects
-				(font
-					(size 1.27 1.27)
-				)
-			)
-		)
-		(property "CurrentEvidence" "INVENTORY UNVERIFIED (E07): inherited 10k PIR pull-up. Cited IMG_2435 establishes R37/R38/R39, but not R33. Physical presence/location and assumed J3.1/J3.2 endpoints remain unverified; retain pending identification, not as a measured value."
-			(at 393.7 353.06 0)
-			(effects
-				(font
-					(size 1.27 1.27)
-				)
-				(hide yes)
-			)
-		)
-		(pin "1"
-		)
-		(pin "2"
-		)
-		(instances
-			(project "PetSafe_1001339"
-				(path "/33a03d59-1679-4e9c-af69-68d086b519af"
-					(reference "R33")
-					(unit 1)
-				)

Commit message: Record Q8 supply continuity and stage S1 contact checks
Parts:
- C6: CurrentEvidence (none) -> C6 is photo-supported in parallel with C5 across H_RF_VDD/G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
- Q8: CurrentEvidence 3724A supports the SIL3724A complementary MOSFET candidate; fitted maker unconfirmed. V113/V115 centre B2/native5 GND is resolved; outer-drain join retains D-E low-resistance evidence. V114 belongs to U2.T2 GND, not Q8. C6 is photo-supported in parallel with C5 as of v0.9.18. Q8 source-supply path remains independently qualified; no current centre-ground conflict. -> 3724A supports the SIL3724A complementary MOSFET candidate; fitted maker unconfirmed. B37 P-F = 1 ohm supports Q8.T2/native2 joining C6.1 on H_RF_VDD. The earlier 10-ohm reading is superseded for the current connection assessment; no fresh probe baseline or stability statement was supplied. V113/V115 centre B2/native5 GND and the outer-drain join retain earlier evidence; V114 belongs to U2.T2. Candidate pin functions, gate drive and operating levels remain unverified.
Changed lines of the file:
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@@
 			)
 		)
+    (property "CurrentEvidence" "C6 is photo-supported in parallel with C5 across H_RF_VDD/GND, after L1. B37 P-F = 1 ohm supports C6 upper pad/model1 joining Q8.T2/native2; no fresh probe baseline or stability statement supplied. This resolves the prior 10-ohm source-path ambiguity for the net reconstruction, not Q8 identity or operation. C6 capacitance remains unknown." (at 259.08 181.61 0)
+      (effects (font (size 1.27 1.27)) (hide yes))
+    )
 		(pin "1"
 		)
@@
 			)
 		)
-		(property "CurrentEvidence" "3724A supports the SIL3724A complementary MOSFET candidate; fitted maker unconfirmed. V113/V115 centre B2/native5 GND is resolved; outer-drain join retains D-E low-resistance evidence. V114 belongs to U2.T2 GND, not Q8. C6 is photo-supported in parallel with C5 as of v0.9.18. Q8 source-supply path remains independently qualified; no current centre-ground conflict."
+		(property "CurrentEvidence" "3724A supports the SIL3724A complementary MOSFET candidate; fitted maker unconfirmed. B37 P-F = 1 ohm supports Q8.T2/native2 joining C6.1 on H_RF_VDD. The earlier 10-ohm reading is superseded for the current connection assessment; no fresh probe baseline or stability statement was supplied. V113/V115 centre B2/native5 GND and the outer-drain join retain earlier evidence; V114 belongs to U2.T2. Candidate pin functions, gate drive and operating levels remain unverified."
 			(at 162.56 231.14 0)
 			(effects

Commit message: Verify S1 contacts and close E05; prepare LED colour checks
Parts:
- Q8: CurrentEvidence 3724A supports the SIL3724A complementary MOSFET candidate; fitted maker unconfirmed. V113/V115 centre B2/native5 GND is resolved; outer-drain join retains D-E low-resistance evidence. V114 belongs to U2.T2 GND, not Q8. C6 is photo-supported in parallel with C5 as of v0.9.18. Q8 source-supply path remains independently qualified; no current centre-ground conflict. -> 3724A supports the SIL3724A complementary MOSFET candidate; fitted maker unconfirmed. B37 P-F = 1 ohm supports Q8.T2/native2 joining C6.1 on H_RF_VDD. The earlier 10-ohm reading is superseded for the current connection assessment; no fresh probe baseline or stability statement was supplied. V113/V115 centre B2/native5 GND and the outer-drain join retain earlier evidence; V114 belongs to U2.T2. Candidate pin functions, gate drive and operating levels remain unverified.
- S1: ContactEvidence (none) -> B38 A-B 1 ohm; B39 C-D 1 ohm; B40 B-D released OL; B41 B-D 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; CurrentEvidence Measured body 6 x 6 x 4 mm plus 2 mm actuator. Stock SW_Pus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 -> B38-B41: A-B and C-D each 1 ohm; B-D released OL and held p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
Changed lines of the file:
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@@
 			)
 		)
-		(property "CurrentEvidence" "Measured body 6 x 6 x 4 mm plus 2 mm actuator. Stock SW_Push has two native nodes: physical TL/TR -> pin1/GND; BL/BR -> pin2/H_BUTTON. R41 reaches J1 VPP. Internal contact pairing and released/pressed behavior remain inferred; the former four-native-pin connector numbering is superseded."
+		(property "CurrentEvidence" "B38-B41: A-B and C-D each 1 ohm; B-D released OL and held pressed 1 ohm. Confirms normally-open S1 with physical TL/TR common on GND (native pin1) and BL/BR common on H_BUTTON (native pin2). Additional A-C OL retained as reported. R41 reaches J1 VPP through the existing 330-ohm path. Contact issue E05 closed; exact footprint fit and the measured 6-mm housing remain separate mechanical qualifications."
 			(at 537.21 60.96 0)
 			(effects
@@
 			)
 		)
+    (property "ContactEvidence" "B38 A-B 1 ohm; B39 C-D 1 ohm; B40 B-D released OL; B41 B-D held pressed 1 ohm. See evidence/s1_contact_results_20261009.json." (at 537.21 60.96 0)
+      (effects (font (size 1.27 1.27)) (hide yes))
+    )
 		(pin "1"
 		)
@@
 		)
 		(mirror x)
-		(property "CurrentEvidence" "3724A supports the SIL3724A complementary MOSFET candidate; fitted maker unconfirmed. V113/V115 centre B2/native5 GND is resolved; outer-drain join retains D-E low-resistance evidence. V114 belongs to U2.T2 GND, not Q8. C6 is photo-supported in parallel with C5 as of v0.9.18. Q8 source-supply path remains independently qualified; no current centre-ground conflict."
+		(property "CurrentEvidence" "3724A supports the SIL3724A complementary MOSFET candidate; fitted maker unconfirmed. B37 P-F = 1 ohm supports Q8.T2/native2 joining C6.1 on H_RF_VDD. The earlier 10-ohm reading is superseded for the current connection assessment; no fresh probe baseline or stability statement was supplied. V113/V115 centre B2/native5 GND and the outer-drain join retain earlier evidence; V114 belongs to U2.T2. Candidate pin functions, gate drive and operating levels remain unverified."
 			(at 162.56 207.01 0)
 			(effects

Commit message: Record LED1 red and green channel mapping; close colour checks
Parts:
- LED1: ColourEvidence (none) -> User B42/B43 colour observations, 2026-10-09; evidence/led1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; ColourMapping (none) -> Native pin1 / R30 / PIC23 = RED; native pin2 / R31 / PIC22 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; CurrentEvidence User confirms square 1.5 x 1.5 mm package containing red an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 -> B42/B43 user diode-mode colour report: photo A-K lights GRE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
Changed lines of the file:
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@@
 			)
 		)
-		(property "CurrentEvidence" "User confirms square 1.5 x 1.5 mm package containing red and green emitters. Four pads and existing board connections retained. Which resistor/PIC channel lights each colour, internal die pairing and exact manufacturer pad numbering remain unconfirmed. No stock land pattern assigned from body size alone."
+		(property "CurrentEvidence" "B42/B43 user diode-mode colour report: photo A-K lights GREEN via R31/PIC22 (LED1 native pin2); B-K lights RED via R30/PIC23 (native pin1). Black probe at grounded K. Both native cathodes 3/4 remain on GND; internal die-to-cathode pairing and manufacturer pad numbers are not established by this in-circuit test. Body 1.5 x 1.5 mm; footprint remains unassigned."
 			(at 231.14 237.49 0)
 			(effects
@@
 			)
 		)
+    (property "ColourMapping" "Native pin1 / R30 / PIC23 = RED; native pin2 / R31 / PIC22 = GREEN" (at 231.14 237.49 0)
+      (effects (font (size 1.27 1.27)) (hide yes))
+    )
+    (property "ColourEvidence" "User B42/B43 colour observations, 2026-10-09; evidence/led1_colour_results_20261009.json" (at 231.14 237.49 0)
+      (effects (font (size 1.27 1.27)) (hide yes))
+    )
 		(pin "1"
 		)
